File: Training_Hardware/Training_Hardware/TIVA.sch (KiCad schematic (older format))
At the start: 8 parts

Commit message: Annotated schematic
Parts:
- gave numbers to parts that had none: 1
Changed lines of the file:
@@
 $EndDescr
 $Comp
-L MRDT_Shields:TM4C129E_Launchpad U?
+L MRDT_Shields:TM4C129E_Launchpad U4
 U 2 1 61497557
 P 3450 3450
-F 0 "U?" H 3700 4700 60  0000 C CNN
+F 0 "U4" H 3700 4700 60  0000 C CNN
 F 1 "TM4C129E_Launchpad" H 3650 4600 60  0000 C CNN
 F 2 "" H 3450 3450 60  0001 C CNN
@@
 $EndComp
 $Comp
-L MRDT_Shields:TM4C129E_Launchpad U?
+L MRDT_Shields:TM4C129E_Launchpad U4
 U 3 1 614996C5
 P 4800 3450
-F 0 "U?" H 5000 3250 60  0000 L CNN
+F 0 "U4" H 5000 3250 60  0000 L CNN
 F 1 "TM4C129E_Launchpad" H 4600 3350 60  0000 L CNN
 F 2 "" H 4800 3450 60  0001 C CNN
@@
 $EndComp
 $Comp
-L MRDT_Shields:TM4C129E_Launchpad U?
+L MRDT_Shields:TM4C129E_Launchpad U4
 U 4 1 6149E2F4
 P 5300 3450
-F 0 "U?" H 5550 4700 60  0000 C CNN
+F 0 "U4" H 5550 4700 60  0000 C CNN
 F 1 "TM4C129E_Launchpad" H 5500 4600 60  0000 C CNN
 F 2 "" H 5300 3450 60  0001 C CNN
@@
 $EndComp
 $Comp
-L MRDT_Shields:TM4C129E_Launchpad U?
+L MRDT_Shields:TM4C129E_Launchpad U4
 U 5 1 614A5B07
 P 2950 5200
-F 0 "U?" H 3100 5000 60  0000 L CNN
+F 0 "U4" H 3100 5000 60  0000 L CNN
 F 1 "TM4C129E_Launchpad" H 2700 5100 60  0000 L CNN
 F 2 "" H 2950 5200 60  0001 C CNN
@@
 $EndComp
 $Comp
-L MRDT_Shields:TM4C129E_Launchpad U?
+L MRDT_Shields:TM4C129E_Launchpad U4
 U 6 1 614A8457
 P 3450 5200
-F 0 "U?" H 3750 6450 60  0000 C CNN
+F 0 "U4" H 3750 6450 60  0000 C CNN
 F 1 "TM4C129E_Launchpad" H 3700 6350 60  0000 C CNN
 F 2 "" H 3450 5200 60  0001 C CNN
@@
 $EndComp
 $Comp
-L MRDT_Shields:TM4C129E_Launchpad U?
+L MRDT_Shields:TM4C129E_Launchpad U4
 U 7 1 614AA8BD
 P 4800 5200
-F 0 "U?" H 4950 5000 60  0000 L CNN
+F 0 "U4" H 4950 5000 60  0000 L CNN
 F 1 "TM4C129E_Launchpad" H 4550 5100 60  0000 L CNN
 F 2 "" H 4800 5200 60  0001 C CNN
@@
 $EndComp
 $Comp
-L MRDT_Shields:TM4C129E_Launchpad U?
+L MRDT_Shields:TM4C129E_Launchpad U4
 U 8 1 614AD240
 P 5300 5200
-F 0 "U?" H 5550 6450 60  0000 C CNN
+F 0 "U4" H 5550 6450 60  0000 C CNN
 F 1 "TM4C129E_Launchpad" H 5550 6350 60  0000 C CNN
 F 2 "" H 5300 5200 60  0001 C CNN
@@
 	3950 2600 3950 2700
 $Comp
-L power:GND #PWR?
+L power:GND #PWR09
 U 1 1 614C375F
 P 3950 2700
-F 0 "#PWR?" H 3950 2450 50  0001 C CNN
+F 0 "#PWR09" H 3950 2450 50  0001 C CNN
 F 1 "GND" H 3955 2527 50  0000 C CNN
 F 2 "" H 3950 2700 50  0001 C CNN
@@
 	5800 2500 5800 2600
 $Comp
-L power:GND #PWR?
+L power:GND #PWR011
 U 1 1 614C40D1
 P 5800 2600
-F 0 "#PWR?" H 5800 2350 50  0001 C CNN
+F 0 "#PWR011" H 5800 2350 50  0001 C CNN
 F 1 "GND" H 5805 2427 50  0000 C CNN
 F 2 "" H 5800 2600 50  0001 C CNN
@@
 	5800 4250 5800 4350
 $Comp
-L power:GND #PWR?
+L power:GND #PWR012
 U 1 1 614C446B
 P 5800 4350
-F 0 "#PWR?" H 5800 4100 50  0001 C CNN
+F 0 "#PWR012" H 5800 4100 50  0001 C CNN
 F 1 "GND" H 5805 4177 50  0000 C CNN
 F 2 "" H 5800 4350 50  0001 C CNN
@@
 	3950 4350 3950 4450
 $Comp
-L power:GND #PWR?
+L power:GND #PWR010
 U 1 1 614C4FB7
 P 3950 4450
-F 0 "#PWR?" H 3950 4200 50  0001 C CNN
+F 0 "#PWR010" H 3950 4200 50  0001 C CNN
 F 1 "GND" H 3955 4277 50  0000 C CNN
 F 2 "" H 3950 4450 50  0001 C CNN
@@
 NoConn ~ 3650 2500
 $Comp
-L MRDT_Shields:TM4C129E_Launchpad U?
+L MRDT_Shields:TM4C129E_Launchpad U4
 U 1 1 61495FA3
 P 2950 3450
-F 0 "U?" H 3100 3250 60  0000 L CNN
+F 0 "U4" H 3100 3250 60  0000 L CNN
 F 1 "TM4C129E_Launchpad" H 2700 3350 60  0000 L CNN
 F 2 "" H 2950 3450 60  0001 C CNN
@@
 	2400 2500 2400 2300
 $Comp
-L power:+3V3 #PWR?
+L power:+3V3 #PWR08
 U 1 1 614E6EDA
 P 2400 2300
-F 0 "#PWR?" H 2400 2150 50  0001 C CNN
+F 0 "#PWR08" H 2400 2150 50  0001 C CNN
 F 1 "+3V3" H 2415 2473 50  0000 C CNN
 F 2 "" H 2400 2300 50  0001 C CNN
