File: Training_Hardware/Training_Hardware/Training_Hardware.sch (KiCad schematic (older format))
At the start: 18 parts

Commit message: Annotated schematic
Parts:
- gave numbers to parts that had none: 16
Changed lines of the file:
@@
 $EndDescr
 $Comp
-L power:+5V #PWR?
+L power:+5V #PWR01
 U 1 1 61465EAA
 P 800 1250
-F 0 "#PWR?" H 800 1100 50  0001 C CNN
+F 0 "#PWR01" H 800 1100 50  0001 C CNN
 F 1 "+5V" H 815 1423 50  0000 C CNN
 F 2 "" H 800 1250 50  0001 C CNN
@@
 	800  1550 800  1250
 $Comp
-L Device:R R?
+L Device:R R1
 U 1 1 6146680B
 P 1150 1550
-F 0 "R?" V 1250 1500 50  0000 L CNN
+F 0 "R1" V 1250 1500 50  0000 L CNN
 F 1 "5.1k" V 1150 1450 50  0000 L CNN
 F 2 "" V 1080 1550 50  0001 C CNN
@@
 $EndComp
 $Comp
-L Device:C C?
+L Device:C C3
 U 1 1 614699BA
 P 1400 2200
-F 0 "C?" H 1515 2246 50  0000 L CNN
+F 0 "C3" H 1515 2246 50  0000 L CNN
 F 1 "0.1μF" H 1515 2155 50  0000 L CNN
 F 2 "" H 1438 2050 50  0001 C CNN
@@
 $EndComp
 $Comp
-L Device:CP1 C?
+L Device:CP1 C6
 U 1 1 6146AE62
 P 2850 2200
-F 0 "C?" H 2965 2246 50  0000 L CNN
+F 0 "C6" H 2965 2246 50  0000 L CNN
 F 1 "10μF 50V" H 2965 2155 50  0000 L CNN
 F 2 "" H 2850 2200 50  0001 C CNN
@@
 $EndComp
 $Comp
-L MRDT_ICs:LT1910 U?
+L MRDT_ICs:LT1910 U3
 U 1 1 6146506C
 P 1800 1950
-F 0 "U?" H 2175 2637 60  0000 C CNN
+F 0 "U3" H 2175 2637 60  0000 C CNN
 F 1 "LT1910" H 2175 2531 60  0000 C CNN
 F 2 "" H 1800 1950 60  0001 C CNN
@@
 	2200 2450 2200 2550
 $Comp
-L power:GND #PWR?
+L power:GND #PWR04
 U 1 1 6146F03B
 P 2200 2550
-F 0 "#PWR?" H 2200 2300 50  0001 C CNN
+F 0 "#PWR04" H 2200 2300 50  0001 C CNN
 F 1 "GND" H 2205 2377 50  0000 C CNN
 F 2 "" H 2200 2550 50  0001 C CNN
@@
 Connection ~ 2850 1550
 $Comp
-L MRDT_Connectors:AndersonPP Conn?
+L MRDT_Connectors:AndersonPP Conn1
 U 4 1 61470ADE
 P 10250 1300
-F 0 "Conn?" H 10222 1347 60  0000 R CNN
+F 0 "Conn1" H 10222 1347 60  0000 R CNN
 F 1 "AndersonPP" H 10222 1453 60  0000 R CNN
 F 2 "" H 10100 750 60  0001 C CNN
@@
 	2850 1250 2850 1550
 $Comp
-L MRDT_Connectors:AndersonPP Conn?
+L MRDT_Connectors:AndersonPP Conn1
 U 1 1 61474817
 P 10250 1900
-F 0 "Conn?" H 10222 1947 60  0000 R CNN
+F 0 "Conn1" H 10222 1947 60  0000 R CNN
 F 1 "AndersonPP" H 10222 2053 60  0000 R CNN
 F 2 "" H 10100 1350 60  0001 C CNN
@@
 $EndComp
 $Comp
-L power:GND #PWR?
+L power:GND #PWR07
 U 1 1 61475E06
 P 9600 2050
-F 0 "#PWR?" H 9600 1800 50  0001 C CNN
+F 0 "#PWR07" H 9600 1800 50  0001 C CNN
 F 1 "GND" H 9605 1877 50  0000 C CNN
 F 2 "" H 9600 2050 50  0001 C CNN
@@
 Connection ~ 3800 2450
 $Comp
-L Device:R R?
+L Device:R R2
 U 1 1 6147B053
 P 3600 2450
-F 0 "R?" V 3500 2450 50  0000 C CNN
+F 0 "R2" V 3500 2450 50  0000 C CNN
 F 1 "3300" V 3600 2450 50  0000 C CNN
 F 2 "" V 3530 2450 50  0001 C CNN
@@
 $EndComp
 $Comp
-L Device:LED D?
+L Device:LED D1
 U 1 1 6147BC08
 P 3200 2450
-F 0 "D?" H 3200 2550 50  0000 C CNN
+F 0 "D1" H 3200 2550 50  0000 C CNN
 F 1 "LED" H 3200 2350 50  0000 C CNN
 F 2 "" H 3200 2450 50  0001 C CNN
@@
 $EndComp
 $Comp
-L Transistor_FET:IRFS4115 Q?
+L Transistor_FET:IRFS4115 Q1
 U 1 1 6147826D
 P 3700 1850
-F 0 "Q?" H 3905 1896 50  0000 L CNN
+F 0 "Q1" H 3905 1896 50  0000 L CNN
 F 1 "IRFS4115" H 3905 1805 50  0000 L CNN
 F 2 "Package_TO_SOT_SMD:TO-263-2" H 3900 1775 50  0001 L CIN
@@
 Connection ~ 2850 2450
 $Comp
-L MRDT_Connectors:AndersonPP Conn?
+L MRDT_Connectors:AndersonPP Conn1
 U 3 1 614843B9
 P 10250 1600
-F 0 "Conn?" H 10222 1647 60  0000 R CNN
+F 0 "Conn1" H 10222 1647 60  0000 R CNN
 F 1 "AndersonPP" H 10222 1753 60  0000 R CNN
 F 2 "" H 10100 1050 60  0001 C CNN
@@
 	1450 1700 1600 1700
 $Comp
-L MRDT_Devices:OKI U?
+L MRDT_Devices:OKI U1
 U 1 1 614ECEC1
 P 1700 3800
-F 0 "U?" H 1750 3750 60  0001 C CNN
+F 0 "U1" H 1750 3750 60  0001 C CNN
 F 1 "OKI" H 1900 4081 60  0000 C CNN
 F 2 "" H 1500 3700 60  0001 C CNN
@@
 $EndComp
 $Comp
-L Device:CP1 C?
+L Device:CP1 C1
 U 1 1 614EDED5
 P 1200 4050
-F 0 "C?" H 1315 4096 50  0000 L CNN
+F 0 "C1" H 1315 4096 50  0000 L CNN
 F 1 "22μF 50V" H 1315 4005 50  0000 L CNN
 F 2 "" H 1200 4050 50  0001 C CNN
@@
 $EndComp
 $Comp
-L Device:C C?
+L Device:C C4
 U 1 1 614EEC63
 P 2500 4050
-F 0 "C?" H 2615 4096 50  0000 L CNN
+F 0 "C4" H 2615 4096 50  0000 L CNN
 F 1 "10μ" H 2615 4005 50  0000 L CNN
 F 2 "" H 2538 3900 50  0001 C CNN
@@
 $EndComp
 $Comp
-L Device:C C?
+L Device:C C7
 U 1 1 614EF0A9
 P 2950 4050
-F 0 "C?" H 3065 4096 50  0000 L CNN
+F 0 "C7" H 3065 4096 50  0000 L CNN
 F 1 "0.1μ" H 3065 4005 50  0000 L CNN
 F 2 "" H 2988 3900 50  0001 C CNN
@@
 Connection ~ 1200 3700
 $Comp
-L power:GND #PWR?
+L power:GND #PWR02
 U 1 1 614F702E
 P 1900 4350
-F 0 "#PWR?" H 1900 4100 50  0001 C CNN
+F 0 "#PWR02" H 1900 4100 50  0001 C CNN
 F 1 "GND" H 1905 4177 50  0000 C CNN
 F 2 "" H 1900 4350 50  0001 C CNN
@@
 $EndComp
 $Comp
-L power:+5V #PWR?
+L power:+5V #PWR05
 U 1 1 614F78D1
 P 3200 3600
-F 0 "#PWR?" H 3200 3450 50  0001 C CNN
+F 0 "#PWR05" H 3200 3450 50  0001 C CNN
 F 1 "+5V" H 3215 3773 50  0000 C CNN
 F 2 "" H 3200 3600 50  0001 C CNN
@@
 	1000 3700 1200 3700
 $Comp
-L MRDT_Devices:OKI U?
+L MRDT_Devices:OKI U2
 U 1 1 61505BC2
 P 1700 5500
-F 0 "U?" H 1750 5450 60  0001 C CNN
+F 0 "U2" H 1750 5450 60  0001 C CNN
 F 1 "OKI" H 1900 5781 60  0000 C CNN
 F 2 "" H 1500 5400 60  0001 C CNN
@@
 $EndComp
 $Comp
-L Device:CP1 C?
+L Device:CP1 C2
 U 1 1 61505BC8
 P 1200 5750
-F 0 "C?" H 1315 5796 50  0000 L CNN
+F 0 "C2" H 1315 5796 50  0000 L CNN
 F 1 "22μF 50V" H 1315 5705 50  0000 L CNN
 F 2 "" H 1200 5750 50  0001 C CNN
@@
 $EndComp
 $Comp
-L Device:C C?
+L Device:C C5
 U 1 1 61505BCE
 P 2500 5750
-F 0 "C?" H 2615 5796 50  0000 L CNN
+F 0 "C5" H 2615 5796 50  0000 L CNN
 F 1 "10μ" H 2615 5705 50  0000 L CNN
 F 2 "" H 2538 5600 50  0001 C CNN
@@
 $EndComp
 $Comp
-L Device:C C?
+L Device:C C8
 U 1 1 61505BD4
 P 2950 5750
-F 0 "C?" H 3065 5796 50  0000 L CNN
+F 0 "C8" H 3065 5796 50  0000 L CNN
 F 1 "0.1μ" H 3065 5705 50  0000 L CNN
 F 2 "" H 2988 5600 50  0001 C CNN
@@
 Connection ~ 1200 5400
 $Comp
-L power:GND #PWR?
+L power:GND #PWR03
 U 1 1 61505BEC
 P 1900 6050
-F 0 "#PWR?" H 1900 5800 50  0001 C CNN
+F 0 "#PWR03" H 1900 5800 50  0001 C CNN
 F 1 "GND" H 1905 5877 50  0000 C CNN
 F 2 "" H 1900 6050 50  0001 C CNN
@@
 	1000 5400 1200 5400
 $Comp
-L power:+3V3 #PWR?
+L power:+3V3 #PWR06
 U 1 1 61507273
 P 3200 5300
-F 0 "#PWR?" H 3200 5150 50  0001 C CNN
+F 0 "#PWR06" H 3200 5150 50  0001 C CNN
 F 1 "+3V3" H 3215 5473 50  0000 C CNN
 F 2 "" H 3200 5300 50  0001 C CNN
