File: Training_Hardware/Training_Hardware/Training_Hardware.sch (KiCad schematic (older format))
At the start: 18 parts

Commit message: created "LT1910" Training circuit
Parts:
- gave numbers to parts that had none: 15
- renumbered Conn?A to Conn?A1, Conn?C to Conn?C1, Conn?D to Conn?D1
Changed lines of the file:
@@
 $EndDescr
 $Comp
-L Amplifier_Current:MAX4081S U?
+L Amplifier_Current:MAX4081S U1
 U 1 1 61465307
 P 3700 2150
-F 0 "U?" H 3750 2728 50  0000 C CNN
+F 0 "U1" H 3750 2728 50  0000 C CNN
 F 1 "\"LT1910\"" H 3750 2637 50  0000 C CNN
 F 2 "" H 4350 1450 50  0001 C CNN
@@
 $EndComp
 $Comp
-L Device:R R?
+L Device:R R1
 U 1 1 6146536D
 P 3050 2050
-F 0 "R?" V 2950 2050 50  0000 C CNN
+F 0 "R1" V 2950 2050 50  0000 C CNN
 F 1 "5.1K" V 3050 2050 50  0000 C CNN
 F 2 "" V 2980 2050 50  0001 C CNN
@@
 	3200 2050 3300 2050
 $Comp
-L Device:C C?
+L Device:C C3
 U 1 1 61465498
 P 3200 2750
-F 0 "C?" H 3315 2796 50  0000 L CNN
+F 0 "C3" H 3315 2796 50  0000 L CNN
 F 1 "0.1uF" H 3315 2705 50  0000 L CNN
 F 2 "" H 3238 2600 50  0001 C CNN
@@
 $EndComp
 $Comp
-L Device:CP1 C?
+L Device:CP1 C8
 U 1 1 61465511
 P 4250 2750
-F 0 "C?" H 4365 2796 50  0000 L CNN
+F 0 "C8" H 4365 2796 50  0000 L CNN
 F 1 "10uF 50V" H 4365 2705 50  0000 L CNN
 F 2 "" H 4250 2750 50  0001 C CNN
@@
 	3200 2900 3200 2950
 $Comp
-L power:+5V #PWR?
+L power:+5V #PWR01
 U 1 1 61465599
 P 2800 1700
-F 0 "#PWR?" H 2800 1550 50  0001 C CNN
+F 0 "#PWR01" H 2800 1550 50  0001 C CNN
 F 1 "+5V" H 2815 1873 50  0000 C CNN
 F 2 "" H 2800 1700 50  0001 C CNN
@@
 	2800 2050 2900 2050
 $Comp
-L power:GND #PWR?
+L power:GND #PWR04
 U 1 1 614656BC
 P 3700 2950
-F 0 "#PWR?" H 3700 2700 50  0001 C CNN
+F 0 "#PWR04" H 3700 2700 50  0001 C CNN
 F 1 "GND" H 3705 2777 50  0000 C CNN
 F 2 "" H 3700 2950 50  0001 C CNN
@@
 	6600 1400 6800 1400
 $Comp
-L Device:Antenna Conn?D
+L Device:Antenna Conn?D1
 U 1 1 614665E9
 P 7000 1400
-F 0 "Conn?D" V 6954 1529 50  0000 L CNN
+F 0 "Conn?D1" V 6954 1529 50  0000 L CNN
 F 1 "\"AndersonPP\"" V 7045 1529 50  0000 L CNN
 F 2 "" H 7000 1400 50  0001 C CNN
@@
 	6600 1800 6800 1800
 $Comp
-L Device:Antenna Conn?A
+L Device:Antenna Conn?A1
 U 1 1 614666D8
 P 7000 1800
-F 0 "Conn?A" V 6954 1929 50  0000 L CNN
+F 0 "Conn?A1" V 6954 1929 50  0000 L CNN
 F 1 "\"AndersonPP\"" V 7045 1929 50  0000 L CNN
 F 2 "" H 7000 1800 50  0001 C CNN
@@
 	6600 1800 6600 1950
 $Comp
-L power:GND #PWR?
+L power:GND #PWR07
 U 1 1 61466AA3
 P 6600 1950
-F 0 "#PWR?" H 6600 1700 50  0001 C CNN
+F 0 "#PWR07" H 6600 1700 50  0001 C CNN
 F 1 "GND" H 6605 1777 50  0000 C CNN
 F 2 "" H 6600 1950 50  0001 C CNN
@@
 $EndComp
 $Comp
-L Connector:XLR3 J?
+L Connector:XLR3 J1
 U 1 1 61467610
 P 5250 2250
-F 0 "J?" V 5204 2477 50  0000 L CNN
+F 0 "J1" V 5204 2477 50  0000 L CNN
 F 1 "XLR3" V 5295 2477 50  0000 L CNN
 F 2 "" H 5250 2250 50  0001 C CNN
@@
 Anderson1
 $Comp
-L Device:R R?
+L Device:R R2
 U 1 1 614681D1
 P 4750 3000
-F 0 "R?" V 4650 3000 50  0000 C CNN
+F 0 "R2" V 4650 3000 50  0000 C CNN
 F 1 "3300" V 4750 3000 50  0000 C CNN
 F 2 "" V 4680 3000 50  0001 C CNN
@@
 $EndComp
 $Comp
-L Device:LED D?
+L Device:LED D1
 U 1 1 61468283
 P 4400 3000
-F 0 "D?" H 4400 3100 50  0000 C CNN
+F 0 "D1" H 4400 3100 50  0000 C CNN
 F 1 "LED" H 4400 2900 50  0000 C CNN
 F 2 "" H 4400 3000 50  0001 C CNN
@@
 Connection ~ 4250 2950
 $Comp
-L Device:Antenna Conn?C
+L Device:Antenna Conn?C1
 U 1 1 61468C3C
 P 7000 1600
-F 0 "Conn?C" V 6954 1729 50  0000 L CNN
+F 0 "Conn?C1" V 6954 1729 50  0000 L CNN
 F 1 "\"AndersonPP\"" V 7045 1729 50  0000 L CNN
 F 2 "" H 7000 1600 50  0001 C CNN
@@
 A1_Signal
 $Comp
-L Transistor_BJT:BUT11 Q?
+L Transistor_BJT:BUT11 Q1
 U 1 1 6146A8C7
 P 2800 3900
-F 0 "Q?" V 3129 3900 50  0000 C CNN
+F 0 "Q1" V 3129 3900 50  0000 C CNN
 F 1 "\"OKI\"" V 3038 3900 50  0000 C CNN
 F 2 "Package_TO_SOT_THT:TO-220-3_Vertical" H 3000 3825 50  0001 L CIN
@@
 $EndComp
 $Comp
-L Device:C C?
+L Device:C C4
 U 1 1 6146A9E5
 P 3400 3950
-F 0 "C?" H 3515 3996 50  0000 L CNN
+F 0 "C4" H 3515 3996 50  0000 L CNN
 F 1 "10uF" H 3450 3850 50  0000 L CNN
 F 2 "" H 3438 3800 50  0001 C CNN
@@
 $EndComp
 $Comp
-L Device:C C?
+L Device:C C6
 U 1 1 6146AA3D
 P 3750 3950
-F 0 "C?" H 3865 3996 50  0000 L CNN
+F 0 "C6" H 3865 3996 50  0000 L CNN
 F 1 ".1uF" H 3800 3850 50  0000 L CNN
 F 2 "" H 3788 3800 50  0001 C CNN
@@
 $EndComp
 $Comp
-L Device:CP1 C?
+L Device:CP1 C1
 U 1 1 6146AA9E
 P 2350 3950
-F 0 "C?" H 2465 3996 50  0000 L CNN
+F 0 "C1" H 2465 3996 50  0000 L CNN
 F 1 "22uF 50V" H 2400 3850 50  0000 L CNN
 F 2 "" H 2350 3950 50  0001 C CNN
@@
 Connection ~ 2350 3800
 $Comp
-L power:GND #PWR?
+L power:GND #PWR02
 U 1 1 6146D134
 P 2800 4100
-F 0 "#PWR?" H 2800 3850 50  0001 C CNN
+F 0 "#PWR02" H 2800 3850 50  0001 C CNN
 F 1 "GND" H 2805 3927 50  0000 C CNN
 F 2 "" H 2800 4100 50  0001 C CNN
@@
 	4100 3800 4100 3700
 $Comp
-L power:+5V #PWR?
+L power:+5V #PWR05
 U 1 1 6146D8F5
 P 4100 3700
-F 0 "#PWR?" H 4100 3550 50  0001 C CNN
+F 0 "#PWR05" H 4100 3550 50  0001 C CNN
 F 1 "+5V" H 4115 3873 50  0000 C CNN
 F 2 "" H 4100 3700 50  0001 C CNN
@@
 PV
 $Comp
-L Transistor_BJT:BUT11 Q?
+L Transistor_BJT:BUT11 Q2
 U 1 1 6146DC4D
 P 2800 4800
-F 0 "Q?" V 3129 4800 50  0000 C CNN
+F 0 "Q2" V 3129 4800 50  0000 C CNN
 F 1 "\"OKI\"" V 3038 4800 50  0000 C CNN
 F 2 "Package_TO_SOT_THT:TO-220-3_Vertical" H 3000 4725 50  0001 L CIN
@@
 $EndComp
 $Comp
-L Device:C C?
+L Device:C C5
 U 1 1 6146DC54
 P 3400 4850
-F 0 "C?" H 3515 4896 50  0000 L CNN
+F 0 "C5" H 3515 4896 50  0000 L CNN
 F 1 "10uF" H 3450 4750 50  0000 L CNN
 F 2 "" H 3438 4700 50  0001 C CNN
@@
 $EndComp
 $Comp
-L Device:C C?
+L Device:C C7
 U 1 1 6146DC5B
 P 3750 4850
-F 0 "C?" H 3865 4896 50  0000 L CNN
+F 0 "C7" H 3865 4896 50  0000 L CNN
 F 1 ".1uF" H 3800 4750 50  0000 L CNN
 F 2 "" H 3788 4700 50  0001 C CNN
@@
 $EndComp
 $Comp
-L Device:CP1 C?
+L Device:CP1 C2
 U 1 1 6146DC62
 P 2350 4850
-F 0 "C?" H 2465 4896 50  0000 L CNN
+F 0 "C2" H 2465 4896 50  0000 L CNN
 F 1 "22uF 50V" H 2400 4750 50  0000 L CNN
 F 2 "" H 2350 4850 50  0001 C CNN
@@
 Connection ~ 2350 4700
 $Comp
-L power:GND #PWR?
+L power:GND #PWR03
 U 1 1 6146DC76
 P 2800 5000
-F 0 "#PWR?" H 2800 4750 50  0001 C CNN
+F 0 "#PWR03" H 2800 4750 50  0001 C CNN
 F 1 "GND" H 2805 4827 50  0000 C CNN
 F 2 "" H 2800 5000 50  0001 C CNN
@@
 PV
 $Comp
-L power:+3V3 #PWR?
+L power:+3V3 #PWR06
 U 1 1 614702A3
 P 4100 4600
-F 0 "#PWR?" H 4100 4450 50  0001 C CNN
+F 0 "#PWR06" H 4100 4450 50  0001 C CNN
 F 1 "+3V3" H 4115 4773 50  0000 C CNN
 F 2 "" H 4100 4600 50  0001 C CNN
