File: Training_Hardware/Training_Hardware/Training_Hardware.sch (KiCad schematic (older format))
At the start: 18 parts

Commit message: LT1910_Changes
Parts:
- gave numbers to parts that had none: 16
Changed lines of the file:
@@
 $EndDescr
 $Comp
-L MRDT_ICs:LT1910 U?
+L MRDT_ICs:LT1910 U1
 U 1 1 614652BB
 P 1700 1700
-F 0 "U?" H 2075 2387 60  0000 C CNN
+F 0 "U1" H 2075 2387 60  0000 C CNN
 F 1 "LT1910" H 2075 2281 60  0000 C CNN
 F 2 "" H 1700 1700 60  0001 C CNN
@@
 $EndComp
 $Comp
-L Device:R R?
+L Device:R R1
 U 1 1 6146B7D6
 P 1150 1300
-F 0 "R?" V 1050 1300 50  0000 C CNN
+F 0 "R1" V 1050 1300 50  0000 C CNN
 F 1 "5.1k" V 1150 1300 50  0000 C CNN
 F 2 "" V 1080 1300 50  0001 C CNN
@@
 	1300 1300 1500 1300
 $Comp
-L power:+5V #PWR?
+L power:+5V #PWR01
 U 1 1 6146EB70
 P 800 1000
-F 0 "#PWR?" H 800 850 50  0001 C CNN
+F 0 "#PWR01" H 800 850 50  0001 C CNN
 F 1 "+5V" H 815 1173 50  0000 C CNN
 F 2 "" H 800 1000 50  0001 C CNN
@@
 	800  1300 1000 1300
 $Comp
-L Device:C C?
+L Device:C C1
 U 1 1 61470AFF
 P 1300 2000
-F 0 "C?" H 1415 2046 50  0000 L CNN
+F 0 "C1" H 1415 2046 50  0000 L CNN
 F 1 "0.1uF" H 1415 1955 50  0000 L CNN
 F 2 "" H 1338 1850 50  0001 C CNN
@@
 	1300 1600 1300 1850
 $Comp
-L power:GND #PWR?
+L power:GND #PWR02
 U 1 1 61474202
 P 2100 2400
-F 0 "#PWR?" H 2100 2150 50  0001 C CNN
+F 0 "#PWR02" H 2100 2150 50  0001 C CNN
 F 1 "GND" H 2105 2227 50  0000 C CNN
 F 2 "" H 2100 2400 50  0001 C CNN
@@
 Connection ~ 2750 1450
 $Comp
-L MRDT_Connectors:AndersonPP Conn?
+L MRDT_Connectors:AndersonPP Conn1
 U 4 1 614779A2
 P 5750 700
-F 0 "Conn?" H 5722 747 60  0000 R CNN
+F 0 "Conn1" H 5722 747 60  0000 R CNN
 F 1 "AndersonPP" H 5722 853 60  0000 R CNN
 F 2 "" H 5600 150 60  0001 C CNN
@@
 	5200 800  5350 800
 $Comp
-L power:GND #PWR?
+L power:GND #PWR07
 U 1 1 6147A963
 P 5100 1450
-F 0 "#PWR?" H 5100 1200 50  0001 C CNN
+F 0 "#PWR07" H 5100 1200 50  0001 C CNN
 F 1 "GND" H 5105 1277 50  0000 C CNN
 F 2 "" H 5100 1450 50  0001 C CNN
@@
 	5100 1300 5100 1450
 $Comp
-L MRDT_Connectors:AndersonPP Conn?
+L MRDT_Connectors:AndersonPP Conn1
 U 1 1 61480536
 P 5750 1200
-F 0 "Conn?" H 5722 1247 60  0000 R CNN
+F 0 "Conn1" H 5722 1247 60  0000 R CNN
 F 1 "AndersonPP" H 5722 1353 60  0000 R CNN
 F 2 "" H 5600 650 60  0001 C CNN
@@
 $EndComp
 $Comp
-L Transistor_FET:IRFS4115 Q?
+L Transistor_FET:IRFS4115 Q1
 U 1 1 61483580
 P 3750 1600
-F 0 "Q?" H 3955 1646 50  0000 L CNN
+F 0 "Q1" H 3955 1646 50  0000 L CNN
 F 1 "IRFS4115" H 3955 1555 50  0000 L CNN
 F 2 "Package_TO_SOT_SMD:TO-263-2" H 3950 1525 50  0001 L CIN
@@
 Anderson1
 $Comp
-L Device:LED D?
+L Device:LED D1
 U 1 1 6148789F
 P 3150 2250
-F 0 "D?" H 3143 2467 50  0000 C CNN
+F 0 "D1" H 3143 2467 50  0000 C CNN
 F 1 "LED" H 3143 2376 50  0000 C CNN
 F 2 "" H 3150 2250 50  0001 C CNN
@@
 	2750 750  2750 1300
 $Comp
-L MRDT_Connectors:AndersonPP Conn?
+L MRDT_Connectors:AndersonPP Conn1
 U 3 1 6148EFAB
 P 5750 950
-F 0 "Conn?" H 5722 997 60  0000 R CNN
+F 0 "Conn1" H 5722 997 60  0000 R CNN
 F 1 "AndersonPP" H 5722 1103 60  0000 R CNN
 F 2 "" H 5600 400 60  0001 C CNN
@@
 	3000 2250 2750 2250
 $Comp
-L Device:CP1 C?
+L Device:CP1 C4
 U 1 1 61471B8E
 P 2750 2000
-F 0 "C?" H 2865 2046 50  0000 L CNN
+F 0 "C4" H 2865 2046 50  0000 L CNN
 F 1 "10uF 50V" H 2865 1955 50  0000 L CNN
 F 2 "" H 2750 2000 50  0001 C CNN
@@
 $EndComp
 $Comp
-L Device:R R?
+L Device:R R2
 U 1 1 6148723F
 P 3550 2250
-F 0 "R?" V 3650 2250 50  0000 C CNN
+F 0 "R2" V 3650 2250 50  0000 C CNN
 F 1 "3300" V 3550 2250 50  0000 C CNN
 F 2 "" V 3480 2250 50  0001 C CNN
@@
 	3850 2250 4050 2250
 $Comp
-L MRDT_Devices:OKI U?
+L MRDT_Devices:OKI U2
 U 1 1 614EA593
 P 1950 3750
-F 0 "U?" H 2000 3700 60  0001 C CNN
+F 0 "U2" H 2000 3700 60  0001 C CNN
 F 1 "OKI" H 2150 4031 60  0000 C CNN
 F 2 "" H 1750 3650 60  0001 C CNN
@@
 $EndComp
 $Comp
-L Device:C C?
+L Device:C C5
 U 1 1 614EA599
 P 2800 3900
-F 0 "C?" H 2550 3950 50  0000 L CNN
+F 0 "C5" H 2550 3950 50  0000 L CNN
 F 1 "10u" H 2500 3850 50  0000 L CNN
 F 2 "" H 2838 3750 50  0001 C CNN
@@
 $EndComp
 $Comp
-L Device:C C?
+L Device:C C7
 U 1 1 614EA59F
 P 3200 3900
-F 0 "C?" H 3315 3946 50  0000 L CNN
+F 0 "C7" H 3315 3946 50  0000 L CNN
 F 1 "0.1u" H 3315 3855 50  0000 L CNN
 F 2 "" H 3238 3750 50  0001 C CNN
@@
 $EndComp
 $Comp
-L Device:CP1 C?
+L Device:CP1 C2
 U 1 1 614EA5A5
 P 1500 3950
-F 0 "C?" H 1615 3996 50  0000 L CNN
+F 0 "C2" H 1615 3996 50  0000 L CNN
 F 1 "22uF 50V" H 1600 3900 50  0000 L CNN
 F 2 "" H 1500 3950 50  0001 C CNN
@@
 	2150 4250 2800 4250
 $Comp
-L power:GND #PWR?
+L power:GND #PWR03
 U 1 1 614EA5BB
 P 2150 4400
-F 0 "#PWR?" H 2150 4150 50  0001 C CNN
+F 0 "#PWR03" H 2150 4150 50  0001 C CNN
 F 1 "GND" H 2155 4227 50  0000 C CNN
 F 2 "" H 2150 4400 50  0001 C CNN
@@
 $EndComp
 $Comp
-L power:+5V #PWR?
+L power:+5V #PWR05
 U 1 1 614EA5C1
 P 3400 3450
-F 0 "#PWR?" H 3400 3300 50  0001 C CNN
+F 0 "#PWR05" H 3400 3300 50  0001 C CNN
 F 1 "+5V" H 3415 3623 50  0000 C CNN
 F 2 "" H 3400 3450 50  0001 C CNN
@@
 Connection ~ 3200 3650
 $Comp
-L MRDT_Devices:OKI U?
+L MRDT_Devices:OKI U3
 U 1 1 614EC30B
 P 1950 5200
-F 0 "U?" H 2000 5150 60  0001 C CNN
+F 0 "U3" H 2000 5150 60  0001 C CNN
 F 1 "OKI" H 2150 5481 60  0000 C CNN
 F 2 "" H 1750 5100 60  0001 C CNN
@@
 $EndComp
 $Comp
-L Device:C C?
+L Device:C C6
 U 1 1 614EC311
 P 2800 5350
-F 0 "C?" H 2550 5400 50  0000 L CNN
+F 0 "C6" H 2550 5400 50  0000 L CNN
 F 1 "10u" H 2500 5300 50  0000 L CNN
 F 2 "" H 2838 5200 50  0001 C CNN
@@
 $EndComp
 $Comp
-L Device:C C?
+L Device:C C8
 U 1 1 614EC317
 P 3200 5350
-F 0 "C?" H 3315 5396 50  0000 L CNN
+F 0 "C8" H 3315 5396 50  0000 L CNN
 F 1 "0.1u" H 3315 5305 50  0000 L CNN
 F 2 "" H 3238 5200 50  0001 C CNN
@@
 $EndComp
 $Comp
-L Device:CP1 C?
+L Device:CP1 C3
 U 1 1 614EC31D
 P 1500 5400
-F 0 "C?" H 1615 5446 50  0000 L CNN
+F 0 "C3" H 1615 5446 50  0000 L CNN
 F 1 "22uF 50V" H 1600 5350 50  0000 L CNN
 F 2 "" H 1500 5400 50  0001 C CNN
@@
 	2150 5700 2800 5700
 $Comp
-L power:GND #PWR?
+L power:GND #PWR04
 U 1 1 614EC333
 P 2150 5850
-F 0 "#PWR?" H 2150 5600 50  0001 C CNN
+F 0 "#PWR04" H 2150 5600 50  0001 C CNN
 F 1 "GND" H 2155 5677 50  0000 C CNN
 F 2 "" H 2150 5850 50  0001 C CNN
@@
 Connection ~ 3200 5100
 $Comp
-L power:+3V3 #PWR?
+L power:+3V3 #PWR06
 U 1 1 614EDA2A
 P 3400 4900
-F 0 "#PWR?" H 3400 4750 50  0001 C CNN
+F 0 "#PWR06" H 3400 4750 50  0001 C CNN
 F 1 "+3V3" H 3415 5073 50  0000 C CNN
 F 2 "" H 3400 4900 50  0001 C CNN
