File: Training_Hardware/Training_Hardware/tiva.sch (KiCad schematic (older format))
At the start: 8 parts

Commit message: LT1910_Changes
Parts:
- gave numbers to parts that had none: 1
Changed lines of the file:
@@
 $EndDescr
 $Comp
-L MRDT_Shields:TM4C129E_Launchpad U?
+L MRDT_Shields:TM4C129E_Launchpad U4
 U 1 1 61496209
 P 1800 2300
-F 0 "U?" H 1000 2950 60  0000 L CNN
+F 0 "U4" H 1000 2950 60  0000 L CNN
 F 1 "TM4C129E_Launchpad" H 550 2800 60  0000 L CNN
 F 2 "" H 1800 2300 60  0001 C CNN
@@
 $EndComp
 $Comp
-L MRDT_Shields:TM4C129E_Launchpad U?
+L MRDT_Shields:TM4C129E_Launchpad U4
 U 2 1 6149E4A3
 P 2300 2300
-F 0 "U?" H 1550 2800 60  0000 C CNN
+F 0 "U4" H 1550 2800 60  0000 C CNN
 F 1 "TM4C129E_Launchpad" H 1500 2700 60  0000 C CNN
 F 2 "" H 2300 2300 60  0001 C CNN
@@
 $EndComp
 $Comp
-L MRDT_Shields:TM4C129E_Launchpad U?
+L MRDT_Shields:TM4C129E_Launchpad U4
 U 3 1 614A446E
 P 4550 2300
-F 0 "U?" H 4750 3650 60  0000 L CNN
+F 0 "U4" H 4750 3650 60  0000 L CNN
 F 1 "TM4C129E_Launchpad" H 4350 3500 60  0000 L CNN
 F 2 "" H 4550 2300 60  0001 C CNN
@@
 $EndComp
 $Comp
-L MRDT_Shields:TM4C129E_Launchpad U?
+L MRDT_Shields:TM4C129E_Launchpad U4
 U 4 1 614A67A0
 P 5050 2300
-F 0 "U?" H 4250 2600 60  0000 C CNN
+F 0 "U4" H 4250 2600 60  0000 C CNN
 F 1 "TM4C129E_Launchpad" H 4200 2500 60  0000 C CNN
 F 2 "" H 5050 2300 60  0001 C CNN
@@
 $EndComp
 $Comp
-L MRDT_Shields:TM4C129E_Launchpad U?
+L MRDT_Shields:TM4C129E_Launchpad U4
 U 5 1 614A8E7F
 P 1800 3600
-F 0 "U?" H 950 4250 60  0000 L CNN
+F 0 "U4" H 950 4250 60  0000 L CNN
 F 1 "TM4C129E_Launchpad" H 550 4050 60  0000 L CNN
 F 2 "" H 1800 3600 60  0001 C CNN
@@
 $EndComp
 $Comp
-L MRDT_Shields:TM4C129E_Launchpad U?
+L MRDT_Shields:TM4C129E_Launchpad U4
 U 6 1 614AC8FA
 P 2300 3600
-F 0 "U?" H 2331 4877 60  0000 C CNN
+F 0 "U4" H 2331 4877 60  0000 C CNN
 F 1 "TM4C129E_Launchpad" H 2331 4771 60  0000 C CNN
 F 2 "" H 2300 3600 60  0001 C CNN
@@
 $EndComp
 $Comp
-L MRDT_Shields:TM4C129E_Launchpad U?
+L MRDT_Shields:TM4C129E_Launchpad U4
 U 7 1 614AEE6D
 P 4550 3550
-F 0 "U?" H 4800 4700 60  0000 L CNN
+F 0 "U4" H 4800 4700 60  0000 L CNN
 F 1 "TM4C129E_Launchpad" H 4450 4700 60  0000 L CNN
 F 2 "" H 4550 3550 60  0001 C CNN
@@
 $EndComp
 $Comp
-L MRDT_Shields:TM4C129E_Launchpad U?
+L MRDT_Shields:TM4C129E_Launchpad U4
 U 8 1 614B22A9
 P 5050 3550
-F 0 "U?" H 4300 4050 60  0000 C CNN
+F 0 "U4" H 4300 4050 60  0000 C CNN
 F 1 "TM4C129E_Launchpad" H 4200 3900 60  0000 C CNN
 F 2 "" H 5050 3550 60  0001 C CNN
@@
 	2700 1450 2700 1600
 $Comp
-L power:GND #PWR?
+L power:GND #PWR09
 U 1 1 614BC98F
 P 2700 1600
-F 0 "#PWR?" H 2700 1350 50  0001 C CNN
+F 0 "#PWR09" H 2700 1350 50  0001 C CNN
 F 1 "GND" H 2705 1427 50  0000 C CNN
 F 2 "" H 2700 1600 50  0001 C CNN
@@
 $EndComp
 $Comp
-L power:GND #PWR?
+L power:GND #PWR011
 U 1 1 614BD101
 P 5550 1550
-F 0 "#PWR?" H 5550 1300 50  0001 C CNN
+F 0 "#PWR011" H 5550 1300 50  0001 C CNN
 F 1 "GND" H 5555 1377 50  0000 C CNN
 F 2 "" H 5550 1550 50  0001 C CNN
@@
 	5600 2600 5600 2750
 $Comp
-L power:GND #PWR?
+L power:GND #PWR012
 U 1 1 614BD417
 P 5600 2750
-F 0 "#PWR?" H 5600 2500 50  0001 C CNN
+F 0 "#PWR012" H 5600 2500 50  0001 C CNN
 F 1 "GND" H 5605 2577 50  0000 C CNN
 F 2 "" H 5600 2750 50  0001 C CNN
@@
 $EndComp
 $Comp
-L power:GND #PWR?
+L power:GND #PWR010
 U 1 1 614BD55E
 P 2700 2950
-F 0 "#PWR?" H 2700 2700 50  0001 C CNN
+F 0 "#PWR010" H 2700 2700 50  0001 C CNN
 F 1 "GND" H 2705 2777 50  0000 C CNN
 F 2 "" H 2700 2950 50  0001 C CNN
@@
 NoConn ~ 2500 1350
 $Comp
-L power:+3V3 #PWR?
+L power:+3V3 #PWR08
 U 1 1 614CE0EB
 P 1400 1100
-F 0 "#PWR?" H 1400 950 50  0001 C CNN
+F 0 "#PWR08" H 1400 950 50  0001 C CNN
 F 1 "+3V3" H 1415 1273 50  0000 C CNN
 F 2 "" H 1400 1100 50  0001 C CNN
