File: Training Hardware/Training_Hardware/Training_Hardware.sch (KiCad schematic (older format))
At the start: 18 parts

Commit message: finished training hardware
Parts:
- gave numbers to parts that had none: 16
Changed lines of the file:
@@
 $EndDescr
 $Comp
-L MRDT_ICs:LT1910 U?
+L MRDT_ICs:LT1910 U3
 U 1 1 6146514A
 P 2250 2600
-F 0 "U?" H 2625 3287 60  0000 C CNN
+F 0 "U3" H 2625 3287 60  0000 C CNN
 F 1 "LT1910" H 2625 3181 60  0000 C CNN
 F 2 "" H 2250 2600 60  0001 C CNN
@@
 $EndComp
 $Comp
-L Device:R R?
+L Device:R R1
 U 1 1 61465BFF
 P 1450 2200
-F 0 "R?" V 1550 2200 50  0000 C CNN
+F 0 "R1" V 1550 2200 50  0000 C CNN
 F 1 "5.1k" V 1450 2200 50  0000 C CNN
 F 2 "" V 1380 2200 50  0001 C CNN
@@
 	1600 2200 2050 2200
 $Comp
-L power:+5V #PWR?
+L power:+5V #PWR01
 U 1 1 61468D4B
 P 1050 1900
-F 0 "#PWR?" H 1050 1750 50  0001 C CNN
+F 0 "#PWR01" H 1050 1750 50  0001 C CNN
 F 1 "+5V" H 1065 2073 50  0000 C CNN
 F 2 "" H 1050 1900 50  0001 C CNN
@@
 	1050 2200 1050 1900
 $Comp
-L Device:C C?
+L Device:C C3
 U 1 1 6146986E
 P 1900 2950
-F 0 "C?" H 2015 2996 50  0000 L CNN
+F 0 "C3" H 2015 2996 50  0000 L CNN
 F 1 "0.1uF" H 2015 2905 50  0000 L CNN
 F 2 "" H 1938 2800 50  0001 C CNN
@@
 $EndComp
 $Comp
-L Device:CP1 C?
+L Device:CP1 C8
 U 1 1 6146A478
 P 3350 2950
-F 0 "C?" H 3465 2996 50  0000 L CNN
+F 0 "C8" H 3465 2996 50  0000 L CNN
 F 1 "10uF 50V" H 3465 2905 50  0000 L CNN
 F 2 "" H 3350 2950 50  0001 C CNN
@@
 	2650 3250 2650 3350
 $Comp
-L power:GND #PWR?
+L power:GND #PWR04
 U 1 1 6146C325
 P 2650 3350
-F 0 "#PWR?" H 2650 3100 50  0001 C CNN
+F 0 "#PWR04" H 2650 3100 50  0001 C CNN
 F 1 "GND" H 2655 3177 50  0000 C CNN
 F 2 "" H 2650 3350 50  0001 C CNN
@@
 	2650 3250 3350 3250
 $Comp
-L SRA_Sensor_Board-rescue:AndersonPP-MRDT_Connectors Conn?
+L SRA_Sensor_Board-rescue:AndersonPP-MRDT_Connectors Conn1
 U 4 1 6146F963
 P 6150 1200
-F 0 "Conn?" H 6122 1247 60  0000 R CNN
+F 0 "Conn1" H 6122 1247 60  0000 R CNN
 F 1 "AndersonPP-MRDT_Connectors" H 6122 1353 60  0000 R CNN
 F 2 "" H 6000 650 60  0001 C CNN
@@
 PV
 $Comp
-L SRA_Sensor_Board-rescue:AndersonPP-MRDT_Connectors Conn?
+L SRA_Sensor_Board-rescue:AndersonPP-MRDT_Connectors Conn1
 U 1 1 61471691
 P 6150 1800
-F 0 "Conn?" H 6122 1847 60  0000 R CNN
+F 0 "Conn1" H 6122 1847 60  0000 R CNN
 F 1 "AndersonPP-MRDT_Connectors" H 6122 1953 60  0000 R CNN
 F 2 "" H 6000 1250 60  0001 C CNN
@@
 $EndComp
 $Comp
-L power:GND #PWR?
+L power:GND #PWR07
 U 1 1 6147259D
 P 5750 2050
-F 0 "#PWR?" H 5750 1800 50  0001 C CNN
+F 0 "#PWR07" H 5750 1800 50  0001 C CNN
 F 1 "GND" H 5755 1877 50  0000 C CNN
 F 2 "" H 5750 2050 50  0001 C CNN
@@
 Anderson1
 $Comp
-L Device:R R?
+L Device:R R2
 U 1 1 6147A5DB
 P 4100 3250
-F 0 "R?" V 4000 3250 50  0000 C CNN
+F 0 "R2" V 4000 3250 50  0000 C CNN
 F 1 "3300" V 4100 3250 50  0000 C CNN
 F 2 "" V 4030 3250 50  0001 C CNN
@@
 $EndComp
 $Comp
-L Device:LED D?
+L Device:LED D1
 U 1 1 6147AD25
 P 3650 3250
-F 0 "D?" H 3650 3350 50  0000 C CNN
+F 0 "D1" H 3650 3350 50  0000 C CNN
 F 1 "LED" H 3650 3150 50  0000 C CNN
 F 2 "" H 3650 3250 50  0001 C CNN
@@
 Connection ~ 3350 3250
 $Comp
-L SRA_Sensor_Board-rescue:AndersonPP-MRDT_Connectors Conn?
+L SRA_Sensor_Board-rescue:AndersonPP-MRDT_Connectors Conn1
 U 3 1 6148280B
 P 6150 1500
-F 0 "Conn?" H 6122 1547 60  0000 R CNN
+F 0 "Conn1" H 6122 1547 60  0000 R CNN
 F 1 "AndersonPP-MRDT_Connectors" H 6122 1653 60  0000 R CNN
 F 2 "" H 6000 950 60  0001 C CNN
@@
 	4250 3250 4350 3250
 $Comp
-L Transistor_FET:IRFS4115 Q?
+L Transistor_FET:IRFS4115 Q1
 U 1 1 614873DF
 P 4250 2500
-F 0 "Q?" H 4455 2546 50  0000 L CNN
+F 0 "Q1" H 4455 2546 50  0000 L CNN
 F 1 "IRFS4115" H 4455 2455 50  0000 L CNN
 F 2 "Package_TO_SOT_SMD:TO-263-2" H 4450 2425 50  0001 L CIN
@@
 	1900 2350 2050 2350
 $Comp
-L MRDT_Devices:OKI U?
+L MRDT_Devices:OKI U2
 U 1 1 614D501C
 P 2000 4600
-F 0 "U?" H 2050 4550 60  0001 C CNN
+F 0 "U2" H 2050 4550 60  0001 C CNN
 F 1 "OKI" H 2200 4881 60  0000 C CNN
 F 2 "" H 1800 4500 60  0001 C CNN
@@
 $EndComp
 $Comp
-L Device:CP1 C?
+L Device:CP1 C2
 U 1 1 614D6F11
 P 1550 4650
-F 0 "C?" H 1665 4696 50  0000 L CNN
+F 0 "C2" H 1665 4696 50  0000 L CNN
 F 1 " 22uF 50V" H 1665 4605 50  0000 L CNN
 F 2 "" H 1550 4650 50  0001 C CNN
@@
 $EndComp
 $Comp
-L Device:C C?
+L Device:C C5
 U 1 1 614D7F7E
 P 2900 4650
-F 0 "C?" H 2700 4700 50  0000 L CNN
+F 0 "C5" H 2700 4700 50  0000 L CNN
 F 1 "10u" H 2650 4600 50  0000 L CNN
 F 2 "" H 2938 4500 50  0001 C CNN
@@
 $EndComp
 $Comp
-L Device:C C?
+L Device:C C7
 U 1 1 614D85FE
 P 3250 4650
-F 0 "C?" H 3365 4696 50  0000 L CNN
+F 0 "C7" H 3365 4696 50  0000 L CNN
 F 1 "0.1u" H 3365 4605 50  0000 L CNN
 F 2 "" H 3288 4500 50  0001 C CNN
@@
 	2200 4950 2200 5050
 $Comp
-L power:GND #PWR?
+L power:GND #PWR03
 U 1 1 614DE85B
 P 2200 5050
-F 0 "#PWR?" H 2200 4800 50  0001 C CNN
+F 0 "#PWR03" H 2200 4800 50  0001 C CNN
 F 1 "GND" H 2205 4877 50  0000 C CNN
 F 2 "" H 2200 5050 50  0001 C CNN
@@
 	1350 4150 1350 4500
 $Comp
-L power:+5V #PWR?
+L power:+5V #PWR06
 U 1 1 614E8106
 P 3600 4250
-F 0 "#PWR?" H 3600 4100 50  0001 C CNN
+F 0 "#PWR06" H 3600 4100 50  0001 C CNN
 F 1 "+5V" H 3615 4423 50  0000 C CNN
 F 2 "" H 3600 4250 50  0001 C CNN
@@
 	3600 4250 3600 4500
 $Comp
-L MRDT_Devices:OKI U?
+L MRDT_Devices:OKI U1
 U 1 1 614EF49F
 P 1800 6400
-F 0 "U?" H 1850 6350 60  0001 C CNN
+F 0 "U1" H 1850 6350 60  0001 C CNN
 F 1 "OKI" H 2000 6681 60  0000 C CNN
 F 2 "" H 1600 6300 60  0001 C CNN
@@
 $EndComp
 $Comp
-L Device:CP1 C?
+L Device:CP1 C1
 U 1 1 614EF4A5
 P 1350 6450
-F 0 "C?" H 1465 6496 50  0000 L CNN
+F 0 "C1" H 1465 6496 50  0000 L CNN
 F 1 " 22uF 50V" H 1465 6405 50  0000 L CNN
 F 2 "" H 1350 6450 50  0001 C CNN
@@
 $EndComp
 $Comp
-L Device:C C?
+L Device:C C4
 U 1 1 614EF4AB
 P 2700 6450
-F 0 "C?" H 2500 6500 50  0000 L CNN
+F 0 "C4" H 2500 6500 50  0000 L CNN
 F 1 "10u" H 2450 6400 50  0000 L CNN
 F 2 "" H 2738 6300 50  0001 C CNN
@@
 $EndComp
 $Comp
-L Device:C C?
+L Device:C C6
 U 1 1 614EF4B1
 P 3050 6450
-F 0 "C?" H 3165 6496 50  0000 L CNN
+F 0 "C6" H 3165 6496 50  0000 L CNN
 F 1 "0.1u" H 3165 6405 50  0000 L CNN
 F 2 "" H 3088 6300 50  0001 C CNN
@@
 	2000 6750 2000 6850
 $Comp
-L power:GND #PWR?
+L power:GND #PWR02
 U 1 1 614EF4C9
 P 2000 6850
-F 0 "#PWR?" H 2000 6600 50  0001 C CNN
+F 0 "#PWR02" H 2000 6600 50  0001 C CNN
 F 1 "GND" H 2005 6677 50  0000 C CNN
 F 2 "" H 2000 6850 50  0001 C CNN
@@
 	1150 5950 1150 6300
 $Comp
-L power:+3V3 #PWR?
+L power:+3V3 #PWR05
 U 1 1 61503FB1
 P 3400 6000
-F 0 "#PWR?" H 3400 5850 50  0001 C CNN
+F 0 "#PWR05" H 3400 5850 50  0001 C CNN
 F 1 "+3V3" H 3415 6173 50  0000 C CNN
 F 2 "" H 3400 6000 50  0001 C CNN
