File: Training Hardware/Training_Hardware/tiva.sch (KiCad schematic (older format))
At the start: 8 parts

Commit message: finished training hardware
Parts:
- gave numbers to parts that had none: 1
Changed lines of the file:
@@
 $EndDescr
 $Comp
-L MRDT_Shields:TM4C129E_Launchpad U?
+L MRDT_Shields:TM4C129E_Launchpad U4
 U 1 1 6148B38E
 P 2100 2250
-F 0 "U?" H 2000 2150 60  0000 L CNN
+F 0 "U4" H 2000 2150 60  0000 L CNN
 F 1 "TM4C129E_Launchpad" H 1650 2000 60  0000 L CNN
 F 2 "" H 2100 2250 60  0001 C CNN
@@
 $EndComp
 $Comp
-L MRDT_Shields:TM4C129E_Launchpad U?
+L MRDT_Shields:TM4C129E_Launchpad U4
 U 2 1 6148DBB0
 P 2600 2250
-F 0 "U?" H 2631 3527 60  0000 C CNN
+F 0 "U4" H 2631 3527 60  0000 C CNN
 F 1 "TM4C129E_Launchpad" H 2631 3421 60  0000 C CNN
 F 2 "" H 2600 2250 60  0001 C CNN
@@
 $EndComp
 $Comp
-L MRDT_Shields:TM4C129E_Launchpad U?
+L MRDT_Shields:TM4C129E_Launchpad U4
 U 3 1 61490A7A
 P 3850 2250
-F 0 "U?" H 3800 2150 60  0000 L CNN
+F 0 "U4" H 3800 2150 60  0000 L CNN
 F 1 "TM4C129E_Launchpad" H 3500 2050 60  0000 L CNN
 F 2 "" H 3850 2250 60  0001 C CNN
@@
 $EndComp
 $Comp
-L MRDT_Shields:TM4C129E_Launchpad U?
+L MRDT_Shields:TM4C129E_Launchpad U4
 U 4 1 61492CC3
 P 4350 2250
-F 0 "U?" H 4381 3527 60  0000 C CNN
+F 0 "U4" H 4381 3527 60  0000 C CNN
 F 1 "TM4C129E_Launchpad" H 4381 3421 60  0000 C CNN
 F 2 "" H 4350 2250 60  0001 C CNN
@@
 $EndComp
 $Comp
-L MRDT_Shields:TM4C129E_Launchpad U?
+L MRDT_Shields:TM4C129E_Launchpad U4
 U 5 1 61495E87
 P 2100 3950
-F 0 "U?" H 2000 3850 60  0000 L CNN
+F 0 "U4" H 2000 3850 60  0000 L CNN
 F 1 "TM4C129E_Launchpad" H 1550 3750 60  0000 L CNN
 F 2 "" H 2100 3950 60  0001 C CNN
@@
 $EndComp
 $Comp
-L MRDT_Shields:TM4C129E_Launchpad U?
+L MRDT_Shields:TM4C129E_Launchpad U4
 U 6 1 61498F64
 P 2600 3950
-F 0 "U?" H 2631 5227 60  0000 C CNN
+F 0 "U4" H 2631 5227 60  0000 C CNN
 F 1 "TM4C129E_Launchpad" H 2631 5121 60  0000 C CNN
 F 2 "" H 2600 3950 60  0001 C CNN
@@
 $EndComp
 $Comp
-L MRDT_Shields:TM4C129E_Launchpad U?
+L MRDT_Shields:TM4C129E_Launchpad U4
 U 7 1 6149B88D
 P 3850 3900
-F 0 "U?" H 3700 3850 60  0000 L CNN
+F 0 "U4" H 3700 3850 60  0000 L CNN
 F 1 "TM4C129E_Launchpad" H 3300 3700 60  0000 L CNN
 F 2 "" H 3850 3900 60  0001 C CNN
@@
 $EndComp
 $Comp
-L MRDT_Shields:TM4C129E_Launchpad U?
+L MRDT_Shields:TM4C129E_Launchpad U4
 U 8 1 6149D82E
 P 4350 3900
-F 0 "U?" H 4381 5177 60  0000 C CNN
+F 0 "U4" H 4381 5177 60  0000 C CNN
 F 1 "TM4C129E_Launchpad" H 4381 5071 60  0000 C CNN
 F 2 "" H 4350 3900 60  0001 C CNN
@@
 	3200 1400 3200 1500
 $Comp
-L power:GND #PWR?
+L power:GND #PWR09
 U 1 1 614C349B
 P 3200 1500
-F 0 "#PWR?" H 3200 1250 50  0001 C CNN
+F 0 "#PWR09" H 3200 1250 50  0001 C CNN
 F 1 "GND" H 3205 1327 50  0000 C CNN
 F 2 "" H 3200 1500 50  0001 C CNN
@@
 	4950 1300 4950 1400
 $Comp
-L power:GND #PWR?
+L power:GND #PWR011
 U 1 1 614C37AF
 P 4950 1400
-F 0 "#PWR?" H 4950 1150 50  0001 C CNN
+F 0 "#PWR011" H 4950 1150 50  0001 C CNN
 F 1 "GND" H 4955 1227 50  0000 C CNN
 F 2 "" H 4950 1400 50  0001 C CNN
@@
 	4950 2950 4950 3050
 $Comp
-L power:GND #PWR?
+L power:GND #PWR012
 U 1 1 614C3CBC
 P 4950 3050
-F 0 "#PWR?" H 4950 2800 50  0001 C CNN
+F 0 "#PWR012" H 4950 2800 50  0001 C CNN
 F 1 "GND" H 4955 2877 50  0000 C CNN
 F 2 "" H 4950 3050 50  0001 C CNN
@@
 	3200 3100 3200 3200
 $Comp
-L power:GND #PWR?
+L power:GND #PWR010
 U 1 1 614C3F1A
 P 3200 3200
-F 0 "#PWR?" H 3200 2950 50  0001 C CNN
+F 0 "#PWR010" H 3200 2950 50  0001 C CNN
 F 1 "GND" H 3205 3027 50  0000 C CNN
 F 2 "" H 3200 3200 50  0001 C CNN
@@
 NoConn ~ 2800 1300
 $Comp
-L power:+3V3 #PWR?
+L power:+3V3 #PWR08
 U 1 1 614D2528
 P 1750 1200
-F 0 "#PWR?" H 1750 1050 50  0001 C CNN
+F 0 "#PWR08" H 1750 1050 50  0001 C CNN
 F 1 "+3V3" H 1765 1373 50  0000 C CNN
 F 2 "" H 1750 1200 50  0001 C CNN
