File: training_hardware/training_hardware.sch (KiCad schematic (older format))
At the start: 18 parts, among them Q1 IRFS4115, U1 LT1910

Commit message: finished naming stuff
Parts:
- gave numbers to parts that had none: 2
- renumbered U1 to U13
Changed lines of the file:
@@
 $EndDescr
 $Comp
-L MRDT_ICs:LT1910 U1
+L MRDT_ICs:LT1910 U13
 U 1 1 614651EC
 P 1750 1650
-F 0 "U1" H 2125 2337 60  0000 C CNN
+F 0 "U13" H 2125 2337 60  0000 C CNN
 F 1 "LT1910" H 2125 2231 60  0000 C CNN
 F 2 "" H 1750 1650 60  0001 C CNN
@@
 A1_signal
 $Comp
-L MRDT_Devices:OKI U?
+L MRDT_Devices:OKI U10
 U 1 1 614DFB18
 P 1850 3250
-F 0 "U?" H 1900 3200 60  0001 C CNN
+F 0 "U10" H 1900 3200 60  0000 C CNN
 F 1 "OKI" H 2050 3531 60  0000 C CNN
 F 2 "" H 1650 3150 60  0001 C CNN
@@
 PV
 $Comp
-L MRDT_Devices:OKI U?
+L MRDT_Devices:OKI U11
 U 1 1 614EBB10
 P 1900 4750
-F 0 "U?" H 1950 4700 60  0001 C CNN
+F 0 "U11" H 1950 4700 60  0000 C CNN
 F 1 "OKI" H 2100 5031 60  0000 C CNN
 F 2 "" H 1700 4650 60  0001 C CNN
